Commit message: Remove parameters for foot link.
We can't identify this link well because it's always in the same spot.

File: examples/Atlas/urdf/planar_quarter_atlas_param.urdf (robot description, URDF)
Before this commit: robot drc_skeleton, 5 links, 4 joints
Links:
- link foot: mass $m__foot -> 4
