Commit message: Add hands to `atlas_chull.urdf`

File: examples/Atlas/urdf/atlas_chull.urdf (robot description, URDF)
Before this commit: robot atlas, 29 links, 28 joints
Links:
- link l_foot: geometry collision mesh filename=meshes/l_foot_chull.wrl scale=1 1 1; collision sphere radius=0
- link l_hand: geometry collision mesh filename=meshes/GRIPPER_OPEN_chull.wrl scale=1 1 1; collision mesh filename=meshes/l_hand_chull.wrl scale=1 1 1
- link r_foot: geometry collision mesh filename=meshes/r_foot_chull.wrl scale=1 1 1; collision sphere radius=0
- link r_hand: geometry collision mesh filename=meshes/GRIPPER_OPEN_chull.wrl scale=1 1 1; collision mesh filename=meshes/r_hand_chull.wrl scale=1 1 1
