Commit message: Torque feasible running for ten steps!
To reproduce run:

```
>> addpath_control
>> cd(fullfile(getDrakePath(),'examples','Atlas','test');
>> options = struct();
>> [sol,r,v,prog] = testRunningPlanner([],1,100,[],options);

In a separate MATLAB instance (to prevent cross-contamination of Atlas
classdefs) run
>> addpath_drake
>> cd(fullfile(getDrakePath(),'examples','Atlas');
>> runAtlasRunning

File: examples/Atlas/urdf/atlas_convex_hull.urdf (robot description, URDF)
Before this commit: robot atlas, 29 links, 28 joints
Joints:
- joint l_leg_aky: limit lower=-1 upper=0.7 effort=350 velocity=12 -> lower=-1 upper=0.7 effort=700 velocity=12
- joint l_leg_kny: limit lower=0 upper=2.38569 effort=220 velocity=12 -> lower=0 upper=2.38569 effort=400 velocity=12
- joint r_leg_aky: limit lower=-1 upper=0.7 effort=350 velocity=12 -> lower=-1 upper=0.7 effort=700 velocity=12
- joint r_leg_kny: limit lower=0 upper=2.38569 effort=220 velocity=12 -> lower=0 upper=2.38569 effort=400 velocity=12

File: examples/Atlas/urdf/atlas_minimal_contact.urdf (robot description, URDF)
Before this commit: robot atlas, 29 links, 28 joints
Joints:
- joint l_leg_aky: limit lower=-1 upper=0.7 effort=350 velocity=12 -> lower=-1 upper=0.7 effort=700 velocity=12
- joint l_leg_kny: limit lower=0 upper=2.38569 effort=220 velocity=12 -> lower=0 upper=2.38569 effort=400 velocity=12
- joint r_leg_aky: limit lower=-1 upper=0.7 effort=350 velocity=12 -> lower=-1 upper=0.7 effort=700 velocity=12
- joint r_leg_kny: limit lower=0 upper=2.38569 effort=220 velocity=12 -> lower=0 upper=2.38569 effort=400 velocity=12
