Commit message: Now the salmon bar is collision free

File: solvers/trajectoryOptimization/test/SalmonBar_rung.urdf (robot description, URDF)
Before this commit: robot SalmonBar_rung, 1 links, 0 joints
Links:
- link salmon_bar_rung: geometry collision box size=0.06 0.05 0.05; visual box size=0.06 0.05 0.05
