Commit message: Switch IRB140 to convex hull collision meshes

File: examples/IRB140/irb_140.urdf (robot description, URDF)
Before this commit: robot IRB140_-_M2004C_Complete_base.SLDASM, 7 links, 6 joints
Links:
- link base_link: geometry visual mesh filename=meshes/base_link.stl
- link link_1: geometry collision mesh filename=meshes/link1_chull.obj; visual mesh filename=meshes/link1.stl
- link link_2: geometry collision mesh filename=meshes/link2_chull.obj; visual mesh filename=meshes/link2.stl
- link link_3: geometry collision mesh filename=meshes/link3_chull.obj; visual mesh filename=meshes/link3.stl
- link link_4: geometry collision mesh filename=meshes/link4_chull.obj; visual mesh filename=meshes/link4.stl
- link link_5: geometry collision mesh filename=meshes/link5_chull.obj; visual mesh filename=meshes/link5.stl
- link link_6: geometry collision mesh filename=meshes/link6_chull.obj; visual mesh filename=meshes/link6.stl
