Commit message: Add iiwa14_mesh_collision.urdf

File: drake/manipulation/models/iiwa_description/urdf/iiwa14.xacro (robot description, xacro)
@@ -38,5 +38,5 @@
           <origin xyz="0 0 0" rpy="0 0 0"/>
           <geometry>
-            <mesh filename="../meshes/collision/link_0.obj"/>
+            <mesh filename="../meshes/collision/link_0_decimated.obj"/>
           </geometry>
           <material name="Grey"/>
@@ -91,5 +91,5 @@
           <origin xyz="0 0 0" rpy="0 0 0"/>
           <geometry>
-            <mesh filename="../meshes/collision/link_1.obj"/>
+            <mesh filename="../meshes/collision/link_1_decimated.obj"/>
           </geometry>
           <material name="Grey"/>
@@ -138,5 +138,5 @@
           <origin xyz="0 0 0" rpy="0 0 0"/>
           <geometry>
-            <mesh filename="../meshes/collision/link_2.obj"/>
+            <mesh filename="../meshes/collision/link_2_decimated.obj"/>
           </geometry>
           <material name="Orange"/>
@@ -185,5 +185,5 @@
           <origin xyz="0 0 0" rpy="0 0 0"/>
           <geometry>
-            <mesh filename="../meshes/collision/link_3.obj"/>
+            <mesh filename="../meshes/collision/link_3_decimated.obj"/>
           </geometry>
           <material name="Grey"/>
@@ -232,5 +232,5 @@
           <origin xyz="0 0 0" rpy="0 0 0"/>
           <geometry>
-            <mesh filename="../meshes/collision/link_4.obj"/>
+            <mesh filename="../meshes/collision/link_4_decimated.obj"/>
           </geometry>
           <material name="Orange"/>
@@ -279,5 +279,5 @@
           <origin xyz="0 0 0" rpy="0 0 0"/>
           <geometry>
-            <mesh filename="../meshes/collision/link_5.obj"/>
+            <mesh filename="../meshes/collision/link_5_decimated.obj"/>
           </geometry>
           <material name="Grey"/>
@@ -326,5 +326,5 @@
           <origin xyz="0 0 0" rpy="0 0 0"/>
           <geometry>
-            <mesh filename="../meshes/collision/link_6.obj"/>
+            <mesh filename="../meshes/collision/link_6_decimated.obj"/>
           </geometry>
           <material name="Orange"/>
@@ -375,5 +375,5 @@
           <origin xyz="0 0 0" rpy="0 0 0"/>
           <geometry>
-            <mesh filename="../meshes/collision/link_7.obj"/>
+            <mesh filename="../meshes/collision/link_7_decimated.obj"/>
           </geometry>
           <material name="Grey"/>
@@ -418,4 +418,15 @@
     <frame name="${robot_name}_frame_ee" link="${robot_name}_link_ee"
            xyz="0.09 0 0" rpy="3.14159265359 0 1.57079632679"/>
+         <collision_filter_group name="${robot_name}_arm">
+           <member link="${robot_name}_link_0"/>
+           <member link="${robot_name}_link_1"/>
+           <member link="${robot_name}_link_2"/>
+           <member link="${robot_name}_link_3"/>
+           <member link="${robot_name}_link_4"/>
+           <member link="${robot_name}_link_5"/>
+           <member link="${robot_name}_link_6"/>
+           <member link="${robot_name}_link_7"/>
+           <ignored_collision_filter_group collision_filter_group="${robot_name}_arm"/>
+         </collision_filter_group>
     <!--Extensions -->
     <xacro:iiwa_gazebo robot_name="${robot_name}" />
