Commit message: [WIP] collision avoidance.

File: drake/manipulation/models/iiwa_description/urdf/iiwa14_primitive_collision.urdf (robot description, URDF)
Before this commit: robot iiwa14, 11 links, 10 joints
Links:
- link iiwa_link_7: geometry collision mesh filename=../meshes/collision/link_7.obj; visual mesh filename=../meshes/collision/link_7.obj
