Commit message: Add min-distance constraints.
Runs, but often gets stuck due to restrictiveness of ee-pose
constraints. Also runs noticably slower.

File: drake/manipulation/models/iiwa_description/urdf/iiwa14_mesh_collision.urdf (robot description, URDF)
Before this commit: robot iiwa14, 11 links, 10 joints
Links:
- link iiwa_link_0: geometry visual mesh filename=../meshes/visual/link_0.obj
- link iiwa_link_1: geometry visual mesh filename=../meshes/visual/link_1.obj

Commit message: [HACK] Add gripper collision geom to iiwa_mesh_collision.urdf

File: drake/manipulation/models/iiwa_description/urdf/iiwa14_mesh_collision.urdf (robot description, URDF)
Before this commit: robot iiwa14, 11 links, 10 joints
Links:
- link iiwa_link_ee: geometry collision box size=0.15, 0.15, 0.10

Commit message: [HACK] Add gripper collision geom to iiwa_mesh_collision.urdf

File: drake/manipulation/models/iiwa_description/urdf/iiwa14_mesh_collision.urdf (robot description, URDF)
Before this commit: robot iiwa14, 11 links, 10 joints
Links:
- link iiwa_link_ee: geometry collision box size=0.15 0.15 0.05

Commit message: [WIP]

File: drake/manipulation/models/iiwa_description/urdf/iiwa14_mesh_collision.urdf (robot description, URDF)
Before this commit: robot iiwa14, 11 links, 10 joints
Links:
- link iiwa_link_0: geometry 

Commit message: Add back in base meshes.

File: drake/manipulation/models/iiwa_description/urdf/iiwa14_mesh_collision.urdf (robot description, URDF)
Before this commit: robot iiwa14, 11 links, 10 joints
Links:
- link iiwa_link_0: geometry collision mesh filename=../meshes/collision/link_0.obj; visual mesh filename=../meshes/visual/link_0.obj
