Commit message: [WIP] Trying to get it working on hardware.

File: drake/examples/kuka_iiwa_arm/models/objects/round_table.urdf (robot description, URDF)
Before this commit: robot round_table, 1 links, 0 joints
Links:
- link table_top: geometry collision cylinder length=1 radius=0.3; visual cylinder length=1 radius=0.3

File: drake/manipulation/models/iiwa_description/urdf/iiwa14_mesh_collision.urdf (robot description, URDF)
Before this commit: robot iiwa14, 11 links, 10 joints
Links:
- link iiwa_link_ee: geometry collision box size=0.15 0.15 0.05; collision sphere radius=0.2
