Commit message: Add tables.

File: manipulation/models/iiwa_description/urdf/iiwa14_spheres_collision.urdf (robot description, URDF)
Before this commit: robot iiwa14, 11 links, 10 joints
Links:
- added link gripper; collision box size=0.0725 0.146 0.049521; collision box size=0.083 0.016 0.02
Joints:
- added joint gripper_joint: type fixed, parent iiwa_link_ee, child gripper, origin xyz=0.13 0 0 rpy=-0.39269908 0 0
