Commit message: [WIP] Add target collision geometry.

File: examples/kuka_iiwa_arm/models/objects/round_table.urdf (robot description, URDF)
Before this commit: robot round_table, 2 links, 1 joints
Links:
- link table_top: geometry collision box size=0.6 0.6 0.017; visual cylinder length=0.017 radius=0.30
